Commit message: fix(urdf): correct mass values in dexhand URDF files
Update mass values in both left and right dexhand URDF files to
reflect accurate measurements. This change ensures the simulation
models are more realistic and align with the physical properties
of the dexhand components.

File: urdf/dexhand021_left_simplified.urdf (robot description, URDF)
Before this commit: robot dexhand021_left_simplified, 26 links, 25 joints
Links:
- link l_f_link1_4: mass 0.511359728172243 -> 0.00511359728172243
- link l_f_link2_4: mass 0.511359728172243 -> 0.00511359728172243
- link l_f_link3_4: mass 0.511359728172243 -> 0.00511359728172243
- link l_f_link4_4: mass 0.511359728172243 -> 0.00511359728172243
- link l_f_link5_4: mass 0.511359728172243 -> 0.00511359728172243

File: urdf/dexhand021_right_simplified.urdf (robot description, URDF)
Before this commit: robot dexhand021_right_simplified, 26 links, 25 joints
Links:
- link r_f_link1_4: mass 0.51136 -> 0.0051136
- link r_f_link2_4: mass 0.51136 -> 0.0051136
- link r_f_link3_4: mass 0.51136 -> 0.0051136
- link r_f_link4_4: mass 0.51136 -> 0.0051136
- link r_f_link5_4: mass 0.51136 -> 0.0051136
