Commit message: fix(urdf): standardize joint limits
Improve the formatting of the URDF files for better readability by
adjusting indentation and line breaks. Add effort and velocity limits
to several joints to enhance simulation accuracy and control. These
changes aim to improve code maintainability and ensure consistent
joint behavior across simulations.

File: urdf/dexhand021_left.urdf (robot description, URDF)
Before this commit: robot dexhand021_left, 58 links, 56 joints
Joints:
- added joint l_f_joint3_3_1: type fixed, parent l_f_link3_3, child l_f_link3_3_1, origin xyz=0 0 0 rpy=0 0 0, axis 0 0 0
- joint l_a_joint1_1: limit lower=0 upper=2.2 -> lower=0 upper=2.2 effort=10 velocity=1.5
- joint l_f_joint1_2: limit lower=0 upper=1.3 -> lower=0 upper=1.3 effort=10 velocity=1.5
- joint l_f_joint1_3: limit lower=0 upper=1.3 -> lower=0 upper=1.3 effort=10 velocity=1.5
- joint l_f_joint1_4: limit lower=0 upper=1.3 -> lower=0 upper=1.3 effort=10 velocity=1.5
- joint l_f_joint2_1: limit lower=0 upper=0.6 -> lower=0 upper=0.6 effort=10 velocity=1.5
- joint l_f_joint2_2: limit lower=0 upper=1.3 -> lower=0 upper=1.3 effort=10 velocity=1.5
- joint l_f_joint2_3: limit lower=0 upper=1.3 effort=0 velocity=0 -> lower=0 upper=1.3 effort=10 velocity=1.5
- joint l_f_joint2_4: limit lower=0 upper=1.3 -> lower=0 upper=1.3 effort=10 velocity=1.5
- joint l_f_joint3_1: limit lower=-0.001 upper=0.001 -> lower=-0.001 upper=0.001 effort=10 velocity=1.5
- joint l_f_joint3_2: limit lower=0 upper=1.3 -> lower=0 upper=1.3 effort=10 velocity=1.5
- joint l_f_joint3_3: limit lower=0 upper=1.3 -> lower=0 upper=1.3 effort=10 velocity=1.5
- joint l_f_joint3_4: limit lower=0 upper=1.3 -> lower=0 upper=1.3 effort=10 velocity=1.5
- joint l_f_joint4_1: limit lower=0 upper=0.6 -> lower=0 upper=0.6 effort=10 velocity=1.5
- joint l_f_joint4_2: limit lower=0 upper=1.3 -> lower=0 upper=1.3 effort=10 velocity=1.5
- joint l_f_joint4_3: limit lower=0 upper=1.3 -> lower=0 upper=1.3 effort=10 velocity=1.5
- joint l_f_joint4_4: limit lower=0 upper=1.3 -> lower=0 upper=1.3 effort=10 velocity=1.5
- joint l_f_joint5_1: limit lower=0 upper=0.6 -> lower=0 upper=0.6 effort=10 velocity=1.5
- joint l_f_joint5_2: limit lower=0 upper=1.3 -> lower=0 upper=1.3 effort=10 velocity=1.5
- joint l_f_joint5_3: limit lower=0 upper=1.3 -> lower=0 upper=1.3 effort=10 velocity=1.5
- joint l_f_joint5_4: limit lower=0 upper=1.3 -> lower=0 upper=1.3 effort=10 velocity=1.5

File: urdf/dexhand021_right.urdf (robot description, URDF)
Before this commit: robot dexhand021_right, 58 links, 57 joints
Joints:
- joint r_f_joint1_1: limit lower=0 upper=2.2 -> lower=0 upper=2.2 effort=10 velocity=1.5
- joint r_f_joint1_2: limit lower=0 upper=1.3 -> lower=0 upper=1.3 effort=10 velocity=1.5
- joint r_f_joint1_3: limit lower=0 upper=1.3 -> lower=0 upper=1.3 effort=10 velocity=1.5
- joint r_f_joint1_4: limit lower=0 upper=1.3 -> lower=0 upper=1.3 effort=10 velocity=1.5
- joint r_f_joint2_1: limit lower=0 upper=0.6 -> lower=0 upper=0.6 effort=10 velocity=1.5
- joint r_f_joint2_2: limit lower=0 upper=1.3 -> lower=0 upper=1.3 effort=10 velocity=1.5
- joint r_f_joint2_3: limit lower=0 upper=1.3 -> lower=0 upper=1.3 effort=10 velocity=1.5
- joint r_f_joint2_4: limit lower=0 upper=1.3 -> lower=0 upper=1.3 effort=10 velocity=1.5
- joint r_f_joint3_1: axis 0 0 0 -> 0 0 1; limit (none) -> lower=-0.001 upper=0.001 effort=10 velocity=1.5; type fixed -> revolute
- joint r_f_joint3_2: limit lower=0 upper=1.3 -> lower=0 upper=1.3 effort=10 velocity=1.5
- joint r_f_joint3_3: limit lower=0 upper=1.3 -> lower=0 upper=1.3 effort=10 velocity=1.5
- joint r_f_joint3_4: limit lower=0 upper=1.3 -> lower=0 upper=1.3 effort=10 velocity=1.5
- joint r_f_joint4_1: limit lower=0 upper=0.6 -> lower=0 upper=0.6 effort=10 velocity=1.5
- joint r_f_joint4_2: limit lower=0 upper=1.3 -> lower=0 upper=1.3 effort=10 velocity=1.5
- joint r_f_joint4_3: limit lower=0 upper=1.3 -> lower=0 upper=1.3 effort=10 velocity=1.5
- joint r_f_joint4_4: limit lower=0 upper=1.3 -> lower=0 upper=1.3 effort=10 velocity=1.5
- joint r_f_joint5_1: limit lower=0 upper=0.6 -> lower=0 upper=0.6 effort=10 velocity=1.5
- joint r_f_joint5_2: limit lower=0 upper=1.3 -> lower=0 upper=1.3 effort=10 velocity=1.5
- joint r_f_joint5_3: limit lower=0 upper=1.3 -> lower=0 upper=1.3 effort=10 velocity=1.5
- joint r_f_joint5_4: limit lower=0 upper=1.3 -> lower=0 upper=1.3 effort=10 velocity=1.5

Commit message: feat(urdf): add fingertips to dexhand models
Add fingertip links and joints to both left and right dexhand URDF
models. This enhancement improves the dexterity and realism of the
robotic hand models by including detailed fingertip representations.
The fingertips are modeled as small spheres with fixed joints,
providing a more accurate simulation of hand movements and interactions.

File: urdf/dexhand021_left.urdf (robot description, URDF)
Before this commit: robot dexhand021_left, 58 links, 57 joints
Links:
- added link l_f_link1_tip, mass 0.001; collision sphere radius=0.002; visual sphere radius=0.002
- added link l_f_link2_tip, mass 0.001; collision sphere radius=0.002; visual sphere radius=0.002
- added link l_f_link3_tip, mass 0.001; collision sphere radius=0.002; visual sphere radius=0.002
- added link l_f_link4_tip, mass 0.001; collision sphere radius=0.002; visual sphere radius=0.002
- added link l_f_link5_tip, mass 0.001; collision sphere radius=0.002; visual sphere radius=0.002
Joints:
- added joint l_f_joint1_tip: type fixed, parent l_f_link1_4, child l_f_link1_tip, origin xyz=0.02 0 0 rpy=0 0 0
- added joint l_f_joint2_tip: type fixed, parent l_f_link2_4, child l_f_link2_tip, origin xyz=0.02 0 0 rpy=0 0 0
- added joint l_f_joint3_tip: type fixed, parent l_f_link3_4, child l_f_link3_tip, origin xyz=0.02 0 0 rpy=0 0 0
- added joint l_f_joint4_tip: type fixed, parent l_f_link4_4, child l_f_link4_tip, origin xyz=0.02 0 0 rpy=0 0 0
- added joint l_f_joint5_tip: type fixed, parent l_f_link5_4, child l_f_link5_tip, origin xyz=0.02 0 0 rpy=0 0 0

File: urdf/dexhand021_right.urdf (robot description, URDF)
Before this commit: robot dexhand021_right, 58 links, 57 joints
Links:
- added link r_f_link1_tip, mass 0.001; collision sphere radius=0.002; visual sphere radius=0.002
- added link r_f_link2_tip, mass 0.001; collision sphere radius=0.002; visual sphere radius=0.002
- added link r_f_link3_tip, mass 0.001; collision sphere radius=0.002; visual sphere radius=0.002
- added link r_f_link4_tip, mass 0.001; collision sphere radius=0.002; visual sphere radius=0.002
- added link r_f_link5_tip, mass 0.001; collision sphere radius=0.002; visual sphere radius=0.002
Joints:
- added joint r_f_joint1_tip: type fixed, parent r_f_link1_4, child r_f_link1_tip, origin xyz=0.02 0 0 rpy=0 0 0
- added joint r_f_joint2_tip: type fixed, parent r_f_link2_4, child r_f_link2_tip, origin xyz=0.02 0 0 rpy=0 0 0
- added joint r_f_joint3_tip: type fixed, parent r_f_link3_4, child r_f_link3_tip, origin xyz=0.02 0 0 rpy=0 0 0
- added joint r_f_joint4_tip: type fixed, parent r_f_link4_4, child r_f_link4_tip, origin xyz=0.02 0 0 rpy=0 0 0
- added joint r_f_joint5_tip: type fixed, parent r_f_link5_4, child r_f_link5_tip, origin xyz=0.02 0 0 rpy=0 0 0

Commit message: feat(models): add simplified STEP and URDF files
Add simplified STEP files for left and right dexhand models to
improve simulation efficiency. Update URDF files to include
simplified models and adjust joint configurations for better
performance. Move existing STL files to a new directory structure
for better organization. Update README to reflect changes and
provide additional resources for model processing.

File: urdf/dexhand021_left.urdf (robot description, URDF)
Before this commit: robot dexhand021_left, 63 links, 62 joints
Joints:
- joint left_base_to_hand: origin xyz=0. 0. -0.17 rpy=0 0 0 -> xyz=0. 0. -0.17 rpy=0 0 1.57

File: urdf/dexhand021_right.urdf (robot description, URDF)
Before this commit: robot dexhand021_right, 63 links, 62 joints
Joints:
- joint right_base_to_hand: origin xyz=0. 0. -0.17 rpy=0 0 0 -> xyz=0. 0. -0.17 rpy=0 0 -1.57
