Commit message: feat(urdf): add density-based inertia calculation
Introduce a utility script `urdf_inertia.py` to calculate and update
inertial properties in URDF files based on mesh density. This enhances
the accuracy of physical simulations by using density maps to assign
appropriate densities to different parts of the model. The script
supports regex-based density mapping and provides a mass report for
verification.

File: urdf/dexhand021_left.urdf (robot description, URDF)
Before this commit: robot dexhand021_left, 63 links, 62 joints
Links:
- link l_f_link1_1: mass 0.0055493 -> 0.005180345836222872; geometry collision mesh filename=../meshes/dexhand021/l_f_link1_1.STL; visual mesh filename=../meshes/dexhand021/l_f_link1_1.STL
- link l_f_link1_2: mass 0.0099742 -> 0.005145873046733005; geometry collision mesh filename=../meshes/dexhand021/l_f_link1_2.STL; visual mesh filename=../meshes/dexhand021/l_f_link1_2.STL
- link l_f_link1_2_1: mass 0.00175 -> 0.001635471969222149; geometry collision mesh filename=../meshes/dexhand021/l_f_link1_2_1.STL; visual mesh filename=../meshes/dexhand021/l_f_link1_2_1.STL
- link l_f_link1_2_2: mass 0.0027191 -> 0.002536590997261413; geometry collision mesh filename=../meshes/dexhand021/l_f_link1_2_2.STL; visual mesh filename=../meshes/dexhand021/l_f_link1_2_2.STL
- link l_f_link1_3: mass 0.0037541 -> 0.003510129470235022; geometry collision mesh filename=../meshes/dexhand021/l_f_link1_3.STL; visual mesh filename=../meshes/dexhand021/l_f_link1_3.STL
- link l_f_link1_3_1: mass 0.00052775 -> 0.0004927439497821334; geometry collision mesh filename=../meshes/dexhand021/l_f_link1_3_1.STL; visual mesh filename=../meshes/dexhand021/l_f_link1_3_1.STL
- link l_f_link1_3_2: mass 0.00099238 -> 0.0009264867224319483; geometry collision mesh filename=../meshes/dexhand021/l_f_link1_3_2.STL; visual mesh filename=../meshes/dexhand021/l_f_link1_3_2.STL
- link l_f_link1_4: mass 0.0046663 -> 0.004357667635534957; geometry collision mesh filename=../meshes/dexhand021/l_f_link1_4.STL; visual mesh filename=../meshes/dexhand021/l_f_link1_4.STL
- link l_f_link1_4_1: mass 0.0031747 -> 0.0003728592379595507; geometry collision mesh filename=../meshes/dexhand021/l_f_link1_4_1.STL; visual mesh filename=../meshes/dexhand021/l_f_link1_4_1.STL
- link l_f_link1_4_2: mass 0.0031747 -> 0.0019468120967671353; geometry collision mesh filename=../meshes/dexhand021/l_f_link1_4_2.STL; visual mesh filename=../meshes/dexhand021/l_f_link1_4_2.STL
- link l_f_link2_1: mass 0.003769 -> 0.0035185790405732886; geometry collision mesh filename=../meshes/dexhand021/l_f_link2_1.STL; visual mesh filename=../meshes/dexhand021/l_f_link2_1.STL
- link l_f_link2_2: mass 0.0053385 -> 0.004989367448655121; geometry collision mesh filename=../meshes/dexhand021/l_f_link2_2.STL; visual mesh filename=../meshes/dexhand021/l_f_link2_2.STL
- link l_f_link2_2_1: mass 0.0010001 -> 0.0009340644343591185; geometry collision mesh filename=../meshes/dexhand021/l_f_link2_2_1.STL; visual mesh filename=../meshes/dexhand021/l_f_link2_2_1.STL
- link l_f_link2_2_2: mass 0.0028758 -> 0.002679962972544191; geometry collision mesh filename=../meshes/dexhand021/l_f_link2_2_2.STL; visual mesh filename=../meshes/dexhand021/l_f_link2_2_2.STL
- link l_f_link2_3: mass 0.0035515 -> 0.003320332898413456; geometry collision mesh filename=../meshes/dexhand021/l_f_link2_3.STL; visual mesh filename=../meshes/dexhand021/l_f_link2_3.STL
- link l_f_link2_3_1: mass 0.00053481 -> 0.0004998303821989263; geometry collision mesh filename=../meshes/dexhand021/l_f_link2_3_1.STL; visual mesh filename=../meshes/dexhand021/l_f_link2_3_1.STL
- link l_f_link2_3_2: mass 0.00099236 -> 0.0009265838824928249; geometry collision mesh filename=../meshes/dexhand021/l_f_link2_3_2.STL; visual mesh filename=../meshes/dexhand021/l_f_link2_3_2.STL
- link l_f_link2_4: mass 0.0046613 -> 0.004352952819276659; geometry collision mesh filename=../meshes/dexhand021/l_f_link2_4.STL; visual mesh filename=../meshes/dexhand021/l_f_link2_4.STL
- link l_f_link2_4_1: mass 0.00041733 -> 0.0003894330192680041; geometry collision mesh filename=../meshes/dexhand021/l_f_link2_4_1.STL; visual mesh filename=../meshes/dexhand021/l_f_link2_4_1.STL
- link l_f_link2_4_2: mass 0.00041733 -> 0.0019468121678303382; geometry collision mesh filename=../meshes/dexhand021/l_f_link2_4_2.STL; visual mesh filename=../meshes/dexhand021/l_f_link2_4_2.STL
- link l_f_link3_1: mass 0.003769 -> 0.0035185790775859407; geometry collision mesh filename=../meshes/dexhand021/l_f_link3_1.STL; visual mesh filename=../meshes/dexhand021/l_f_link3_1.STL
- link l_f_link3_2: mass 0.0053385 -> 0.004989367448655343; geometry collision mesh filename=../meshes/dexhand021/l_f_link3_2.STL; visual mesh filename=../meshes/dexhand021/l_f_link3_2.STL
- link l_f_link3_2_1: mass 0.0010001 -> 0.0009340644343591204; geometry collision mesh filename=../meshes/dexhand021/l_f_link3_2_1.STL; visual mesh filename=../meshes/dexhand021/l_f_link3_2_1.STL
- link l_f_link3_2_2: mass 0.0028758 -> 0.0026799629725441833; geometry collision mesh filename=../meshes/dexhand021/l_f_link3_2_2.STL; visual mesh filename=../meshes/dexhand021/l_f_link3_2_2.STL
- link l_f_link3_3: mass 0.0035515 -> 0.0033203328984136053; geometry collision mesh filename=../meshes/dexhand021/l_f_link3_3.STL; visual mesh filename=../meshes/dexhand021/l_f_link3_3.STL
- link l_f_link3_3_1: mass 0.0010001 -> 0.0004998303821669769; geometry collision mesh filename=../meshes/dexhand021/l_f_link3_3_1.STL; visual mesh filename=../meshes/dexhand021/l_f_link3_3_1.STL
- link l_f_link3_3_2: mass 0.00099236 -> 0.0009265838824928253; geometry collision mesh filename=../meshes/dexhand021/l_f_link3_3_2.STL; visual mesh filename=../meshes/dexhand021/l_f_link3_3_2.STL
- link l_f_link3_4: mass 0.0046613 -> 0.004352952819355013; geometry collision mesh filename=../meshes/dexhand021/l_f_link3_4.STL; visual mesh filename=../meshes/dexhand021/l_f_link3_4.STL
- link l_f_link3_4_1: mass 0.00041733 -> 0.00038943301930773646; geometry collision mesh filename=../meshes/dexhand021/l_f_link3_4_1.STL; visual mesh filename=../meshes/dexhand021/l_f_link3_4_1.STL
- link l_f_link3_4_2: mass 0.00041733 -> 0.0019468121676849014; geometry collision mesh filename=../meshes/dexhand021/l_f_link3_4_2.STL; visual mesh filename=../meshes/dexhand021/l_f_link3_4_2.STL
- link l_f_link4_1: mass 0.003769 -> 0.003518579078981058; geometry collision mesh filename=../meshes/dexhand021/l_f_link4_1.STL; visual mesh filename=../meshes/dexhand021/l_f_link4_1.STL
- link l_f_link4_2: mass 0.0053385 -> 0.004989367448655342; geometry collision mesh filename=../meshes/dexhand021/l_f_link4_2.STL; visual mesh filename=../meshes/dexhand021/l_f_link4_2.STL
- link l_f_link4_2_1: mass 0.0010001 -> 0.0009340644343591187; geometry collision mesh filename=../meshes/dexhand021/l_f_link4_2_1.STL; visual mesh filename=../meshes/dexhand021/l_f_link4_2_1.STL
- link l_f_link4_2_2: mass 0.0028758 -> 0.002679962972544182; geometry collision mesh filename=../meshes/dexhand021/l_f_link4_2_2.STL; visual mesh filename=../meshes/dexhand021/l_f_link4_2_2.STL
- link l_f_link4_3: mass 0.0035515 -> 0.0033203328984136053; geometry collision mesh filename=../meshes/dexhand021/l_f_link4_3.STL; visual mesh filename=../meshes/dexhand021/l_f_link4_3.STL
- link l_f_link4_3_1: mass 0.00053481 -> 0.0004998303821989261; geometry collision mesh filename=../meshes/dexhand021/l_f_link4_3_1.STL; visual mesh filename=../meshes/dexhand021/l_f_link4_3_1.STL
- link l_f_link4_3_2: mass 0.00099236 -> 0.0009265838824928249; geometry collision mesh filename=../meshes/dexhand021/l_f_link4_3_2.STL; visual mesh filename=../meshes/dexhand021/l_f_link4_3_2.STL
- link l_f_link4_4: mass 0.0046613 -> 0.004352952819355011; geometry collision mesh filename=../meshes/dexhand021/l_f_link4_4.STL; visual mesh filename=../meshes/dexhand021/l_f_link4_4.STL
- link l_f_link4_4_1: mass 0.00041733 -> 0.00038943301930773673; geometry collision mesh filename=../meshes/dexhand021/l_f_link4_4_1.STL; visual mesh filename=../meshes/dexhand021/l_f_link4_4_1.STL
- link l_f_link4_4_2: mass 0.00041733 -> 0.0019468121676848738; geometry collision mesh filename=../meshes/dexhand021/l_f_link4_4_2.STL; visual mesh filename=../meshes/dexhand021/l_f_link4_4_2.STL
- link l_f_link5_1: mass 0.003769 -> 0.0035185790783407995; geometry collision mesh filename=../meshes/dexhand021/l_f_link5_1.STL; visual mesh filename=../meshes/dexhand021/l_f_link5_1.STL
- link l_f_link5_2: mass 0.0053385 -> 0.004989367448655121; geometry collision mesh filename=../meshes/dexhand021/l_f_link5_2.STL; visual mesh filename=../meshes/dexhand021/l_f_link5_2.STL
- link l_f_link5_2_1: mass 0.0010001 -> 0.0009340644343591205; geometry collision mesh filename=../meshes/dexhand021/l_f_link5_2_1.STL; visual mesh filename=../meshes/dexhand021/l_f_link5_2_1.STL
- link l_f_link5_2_2: mass 0.0028758 -> 0.002679962972544193; geometry collision mesh filename=../meshes/dexhand021/l_f_link5_2_2.STL; visual mesh filename=../meshes/dexhand021/l_f_link5_2_2.STL
- link l_f_link5_3: mass 0.0035515 -> 0.003320332898413456; geometry collision mesh filename=../meshes/dexhand021/l_f_link5_3.STL; visual mesh filename=../meshes/dexhand021/l_f_link5_3.STL
- link l_f_link5_3_1: mass 0.00053481 -> 0.0004998303821669769; geometry collision mesh filename=../meshes/dexhand021/l_f_link5_3_1.STL; visual mesh filename=../meshes/dexhand021/l_f_link5_3_1.STL
- link l_f_link5_3_2: mass 0.00099236 -> 0.0009265838824928253; geometry collision mesh filename=../meshes/dexhand021/l_f_link5_3_2.STL; visual mesh filename=../meshes/dexhand021/l_f_link5_3_2.STL
- link l_f_link5_4: mass 0.0046613 -> 0.00435295285508909; geometry collision mesh filename=../meshes/dexhand021/l_f_link5_4.STL; visual mesh filename=../meshes/dexhand021/l_f_link5_4.STL
- link l_f_link5_4_1: mass 0.00041733 -> 0.0003894330192680038; geometry collision mesh filename=../meshes/dexhand021/l_f_link5_4_1.STL; visual mesh filename=../meshes/dexhand021/l_f_link5_4_1.STL
- link l_f_link5_4_2: mass 0.00041733 -> 0.0019468121678303657; geometry collision mesh filename=../meshes/dexhand021/l_f_link5_4_2.STL; visual mesh filename=../meshes/dexhand021/l_f_link5_4_2.STL
- link l_p_link0: mass 0.37509 -> 0.4582127297726252; geometry collision mesh filename=../meshes/dexhand021/l_p_link0.STL; visual mesh filename=../meshes/dexhand021/l_p_link0.STL
- link l_p_link1: mass 0.027206 -> 0.08402879470191237; geometry collision mesh filename=../meshes/dexhand021/l_p_link1.STL; visual mesh filename=../meshes/dexhand021/l_p_link1.STL
- link l_p_link2: mass 0.0256 -> 0.07899885001313191; geometry collision mesh filename=../meshes/dexhand021/l_p_link2.STL; visual mesh filename=../meshes/dexhand021/l_p_link2.STL
- link l_p_link3: mass 0.014275 -> 0.04403763346723259; geometry collision mesh filename=../meshes/dexhand021/l_p_link3.STL; visual mesh filename=../meshes/dexhand021/l_p_link3.STL
- link l_p_link4: mass 0.026683 -> 0.08225994389583667; geometry collision mesh filename=../meshes/dexhand021/l_p_link4.STL; visual mesh filename=../meshes/dexhand021/l_p_link4.STL
- link l_p_link5: mass 0.0073198 -> 0.022514206360667064; geometry collision mesh filename=../meshes/dexhand021/l_p_link5.STL; visual mesh filename=../meshes/dexhand021/l_p_link5.STL
- link l_p_link6: mass 0.036656 -> 0.11250344206877806; geometry collision mesh filename=../meshes/dexhand021/l_p_link6.STL; visual mesh filename=../meshes/dexhand021/l_p_link6.STL

File: urdf/dexhand021_left_simplified.urdf (robot description, URDF)
Before this commit: robot dexhand021_left_simplified, 26 links, 25 joints
Links:
- link l_f_link1_1: mass 0.0055493 -> 0.004409652627263485; geometry collision mesh filename=../meshes/dexhand021_simplified/l_f_link1_1.STL; visual mesh filename=../meshes/dexhand021_simplified/l_f_link1_1.STL
- link l_f_link1_2: mass 0.0124624337931872 -> 0.009951630175659748; geometry collision mesh filename=../meshes/dexhand021_simplified/l_f_link1_2.STL; visual mesh filename=../meshes/dexhand021_simplified/l_f_link1_2.STL
- link l_f_link1_3: mass 0.00572598940663931 -> 0.004572753893586383; geometry collision mesh filename=../meshes/dexhand021_simplified/l_f_link1_3.STL; visual mesh filename=../meshes/dexhand021_simplified/l_f_link1_3.STL
- link l_f_link1_4: mass 0.00511359728172243 -> 0.0061582385243810385; geometry collision mesh filename=../meshes/dexhand021_simplified/l_f_link1_4.STL; visual mesh filename=../meshes/dexhand021_simplified/l_f_link1_4.STL
- link l_f_link2_1: mass 0.00512730147699983 -> 0.004097010287465458; geometry collision mesh filename=../meshes/dexhand021_simplified/l_f_link2_1.STL; visual mesh filename=../meshes/dexhand021_simplified/l_f_link2_1.STL
- link l_f_link2_2: mass 0.011802504617909 -> 0.009428301114189446; geometry collision mesh filename=../meshes/dexhand021_simplified/l_f_link2_2.STL; visual mesh filename=../meshes/dexhand021_simplified/l_f_link2_2.STL
- link l_f_link2_3: mass 0.0057259887397435 -> 0.004572753788929435; geometry collision mesh filename=../meshes/dexhand021_simplified/l_f_link2_3.STL; visual mesh filename=../meshes/dexhand021_simplified/l_f_link2_3.STL
- link l_f_link2_4: mass 0.00511359728172243 -> 0.00615823855422499; geometry collision mesh filename=../meshes/dexhand021_simplified/l_f_link2_4.STL; visual mesh filename=../meshes/dexhand021_simplified/l_f_link2_4.STL
- link l_f_link3_1: mass 0.00512729840681515 -> 0.004097008090990198; geometry collision mesh filename=../meshes/dexhand021_simplified/l_f_link3_1.STL; visual mesh filename=../meshes/dexhand021_simplified/l_f_link3_1.STL
- link l_f_link3_2: mass 0.011802504617909 -> 0.009428301114189446; geometry collision mesh filename=../meshes/dexhand021_simplified/l_f_link3_2.STL; visual mesh filename=../meshes/dexhand021_simplified/l_f_link3_2.STL
- link l_f_link3_3: mass 0.00572598873974363 -> 0.004572753789108405; geometry collision mesh filename=../meshes/dexhand021_simplified/l_f_link3_3.STL; visual mesh filename=../meshes/dexhand021_simplified/l_f_link3_3.STL
- link l_f_link3_4: mass 0.00511359728172243 -> 0.00615823855422499; geometry collision mesh filename=../meshes/dexhand021_simplified/l_f_link3_4.STL; visual mesh filename=../meshes/dexhand021_simplified/l_f_link3_4.STL
- link l_f_link4_1: mass 0.00512729933180569 -> 0.004097008849009738; geometry collision mesh filename=../meshes/dexhand021_simplified/l_f_link4_1.STL; visual mesh filename=../meshes/dexhand021_simplified/l_f_link4_1.STL
- link l_f_link4_2: mass 0.0118025067643813 -> 0.009428301114189446; geometry collision mesh filename=../meshes/dexhand021_simplified/l_f_link4_2.STL; visual mesh filename=../meshes/dexhand021_simplified/l_f_link4_2.STL
- link l_f_link4_3: mass 0.00572598873974366 -> 0.004572753788921786; geometry collision mesh filename=../meshes/dexhand021_simplified/l_f_link4_3.STL; visual mesh filename=../meshes/dexhand021_simplified/l_f_link4_3.STL
- link l_f_link4_4: mass 0.00511359728172243 -> 0.00615823855422499; geometry collision mesh filename=../meshes/dexhand021_simplified/l_f_link4_4.STL; visual mesh filename=../meshes/dexhand021_simplified/l_f_link4_4.STL
- link l_f_link5_1: mass 0.00512729994652864 -> 0.004097005770491854; geometry collision mesh filename=../meshes/dexhand021_simplified/l_f_link5_1.STL; visual mesh filename=../meshes/dexhand021_simplified/l_f_link5_1.STL
- link l_f_link5_2: mass 0.0118025067643815 -> 0.009428301114189446; geometry collision mesh filename=../meshes/dexhand021_simplified/l_f_link5_2.STL; visual mesh filename=../meshes/dexhand021_simplified/l_f_link5_2.STL
- link l_f_link5_3: mass 0.00572598873974358 -> 0.004572753788933973; geometry collision mesh filename=../meshes/dexhand021_simplified/l_f_link5_3.STL; visual mesh filename=../meshes/dexhand021_simplified/l_f_link5_3.STL
- link l_f_link5_4: mass 0.00511359728172243 -> 0.00615823855422499; geometry collision mesh filename=../meshes/dexhand021_simplified/l_f_link5_4.STL; visual mesh filename=../meshes/dexhand021_simplified/l_f_link5_4.STL
- link left_hand_base: mass 0.37509 -> 0.8839820474170381; geometry collision mesh filename=../meshes/dexhand021_simplified/left_hand_base.STL; visual mesh filename=../meshes/dexhand021_simplified/left_hand_base.STL
