Commit message: feat(urdf): add density-based inertia calculation
Introduce a utility script `urdf_inertia.py` to calculate and update
inertial properties in URDF files based on mesh density. This enhances
the accuracy of physical simulations by using density maps to assign
appropriate densities to different parts of the model. The script
supports regex-based density mapping and provides a mass report for
verification.

File: urdf/dexhand021_right.urdf (robot description, URDF)
Before this commit: robot dexhand021_right, 63 links, 62 joints
Links:
- link r_f_link1_1: mass 0.0055494 -> 0.005180345914026771; geometry collision mesh filename=../meshes/dexhand021/r_f_link1_1.STL; visual mesh filename=../meshes/dexhand021/r_f_link1_1.STL
- link r_f_link1_2: mass 0.0055051 -> 0.005145873046732899; geometry collision mesh filename=../meshes/dexhand021/r_f_link1_2.STL; visual mesh filename=../meshes/dexhand021/r_f_link1_2.STL
- link r_f_link1_2_1: mass 0.00175 -> 0.0016354719692142122; geometry collision mesh filename=../meshes/dexhand021/r_f_link1_2_1.STL; visual mesh filename=../meshes/dexhand021/r_f_link1_2_1.STL
- link r_f_link1_2_2: mass 0.0027191 -> 0.002536590997261413; geometry collision mesh filename=../meshes/dexhand021/r_f_link1_2_2.STL; visual mesh filename=../meshes/dexhand021/r_f_link1_2_2.STL
- link r_f_link1_3: mass 0.0037541 -> 0.003510129470234603; geometry collision mesh filename=../meshes/dexhand021/r_f_link1_3.STL; visual mesh filename=../meshes/dexhand021/r_f_link1_3.STL
- link r_f_link1_3_1: mass 0.00052776 -> 0.0004927439497821333; geometry collision mesh filename=../meshes/dexhand021/r_f_link1_3_1.STL; visual mesh filename=../meshes/dexhand021/r_f_link1_3_1.STL
- link r_f_link1_3_2: mass 0.00099237 -> 0.0009264867224319483; geometry collision mesh filename=../meshes/dexhand021/r_f_link1_3_2.STL; visual mesh filename=../meshes/dexhand021/r_f_link1_3_2.STL
- link r_f_link1_4: mass 0.0046663 -> 0.00435766768406691; geometry collision mesh filename=../meshes/dexhand021/r_f_link1_4.STL; visual mesh filename=../meshes/dexhand021/r_f_link1_4.STL
- link r_f_link1_4_1: mass 0.0031747 -> 0.00037285923791626445; geometry collision mesh filename=../meshes/dexhand021/r_f_link1_4_1.STL; visual mesh filename=../meshes/dexhand021/r_f_link1_4_1.STL
- link r_f_link1_4_2: mass 0.0031747 -> 0.0019468120969125988; geometry collision mesh filename=../meshes/dexhand021/r_f_link1_4_2.STL; visual mesh filename=../meshes/dexhand021/r_f_link1_4_2.STL
- link r_f_link2_1: mass 0.003769 -> 0.0035185790867912825; geometry collision mesh filename=../meshes/dexhand021/r_f_link2_1.STL; visual mesh filename=../meshes/dexhand021/r_f_link2_1.STL
- link r_f_link2_2: mass 0.0053385 -> 0.00498936744865468; geometry collision mesh filename=../meshes/dexhand021/r_f_link2_2.STL; visual mesh filename=../meshes/dexhand021/r_f_link2_2.STL
- link r_f_link2_2_1: mass 0.0010001 -> 0.0009340644343559288; geometry collision mesh filename=../meshes/dexhand021/r_f_link2_2_1.STL; visual mesh filename=../meshes/dexhand021/r_f_link2_2_1.STL
- link r_f_link2_2_2: mass 0.0028758 -> 0.00267996297249627; geometry collision mesh filename=../meshes/dexhand021/r_f_link2_2_2.STL; visual mesh filename=../meshes/dexhand021/r_f_link2_2_2.STL
- link r_f_link2_3: mass 0.0035515 -> 0.003320332898413509; geometry collision mesh filename=../meshes/dexhand021/r_f_link2_3.STL; visual mesh filename=../meshes/dexhand021/r_f_link2_3.STL
- link r_f_link2_3_1: mass 0.00053481 -> 0.0004998303821989283; geometry collision mesh filename=../meshes/dexhand021/r_f_link2_3_1.STL; visual mesh filename=../meshes/dexhand021/r_f_link2_3_1.STL
- link r_f_link2_3_2: mass 0.00099236 -> 0.0009265838824928239; geometry collision mesh filename=../meshes/dexhand021/r_f_link2_3_2.STL; visual mesh filename=../meshes/dexhand021/r_f_link2_3_2.STL
- link r_f_link2_4: mass 0.0046613 -> 0.004352952819365211; geometry collision mesh filename=../meshes/dexhand021/r_f_link2_4.STL; visual mesh filename=../meshes/dexhand021/r_f_link2_4.STL
- link r_f_link2_4_1: mass 0.00041733 -> 0.00038943301930674843; geometry collision mesh filename=../meshes/dexhand021/r_f_link2_4_1.STL; visual mesh filename=../meshes/dexhand021/r_f_link2_4_1.STL
- link r_f_link2_4_2: mass 0.0110157 -> 0.0019468121675446145; geometry collision mesh filename=../meshes/dexhand021/r_f_link2_4_2.STL; visual mesh filename=../meshes/dexhand021/r_f_link2_4_2.STL
- link r_f_link3_1: mass 0.003769 -> 0.003518579086791124; geometry collision mesh filename=../meshes/dexhand021/r_f_link3_1.STL; visual mesh filename=../meshes/dexhand021/r_f_link3_1.STL
- link r_f_link3_2: mass 0.0053385 -> 0.004989367448661263; geometry collision mesh filename=../meshes/dexhand021/r_f_link3_2.STL; visual mesh filename=../meshes/dexhand021/r_f_link3_2.STL
- link r_f_link3_2_1: mass 0.0010001 -> 0.0009340644343708481; geometry collision mesh filename=../meshes/dexhand021/r_f_link3_2_1.STL; visual mesh filename=../meshes/dexhand021/r_f_link3_2_1.STL
- link r_f_link3_2_2: mass 0.0028758 -> 0.0026799629725441426; geometry collision mesh filename=../meshes/dexhand021/r_f_link3_2_2.STL; visual mesh filename=../meshes/dexhand021/r_f_link3_2_2.STL
- link r_f_link3_3: mass 0.0035515 -> 0.0033203328984138664; geometry collision mesh filename=../meshes/dexhand021/r_f_link3_3.STL; visual mesh filename=../meshes/dexhand021/r_f_link3_3.STL
- link r_f_link3_3_1: mass 0.00053481 -> 0.000499830382198927; geometry collision mesh filename=../meshes/dexhand021/r_f_link3_3_1.STL; visual mesh filename=../meshes/dexhand021/r_f_link3_3_1.STL
- link r_f_link3_3_2: mass 0.00099236 -> 0.0009265838824928244; geometry collision mesh filename=../meshes/dexhand021/r_f_link3_3_2.STL; visual mesh filename=../meshes/dexhand021/r_f_link3_3_2.STL
- link r_f_link3_4: mass 0.0046613 -> 0.00435295281947875; geometry collision mesh filename=../meshes/dexhand021/r_f_link3_4.STL; visual mesh filename=../meshes/dexhand021/r_f_link3_4.STL
- link r_f_link3_4_1: mass 0.00041733 -> 0.00038943301930674805; geometry collision mesh filename=../meshes/dexhand021/r_f_link3_4_1.STL; visual mesh filename=../meshes/dexhand021/r_f_link3_4_1.STL
- link r_f_link3_4_2: mass 0.0110157 -> 0.0019468121669157683; geometry collision mesh filename=../meshes/dexhand021/r_f_link3_4_2.STL; visual mesh filename=../meshes/dexhand021/r_f_link3_4_2.STL
- link r_f_link4_1: mass 0.003769 -> 0.003518579086791169; geometry collision mesh filename=../meshes/dexhand021/r_f_link4_1.STL; visual mesh filename=../meshes/dexhand021/r_f_link4_1.STL
- link r_f_link4_2: mass 0.0053385 -> 0.004989367448655343; geometry collision mesh filename=../meshes/dexhand021/r_f_link4_2.STL; visual mesh filename=../meshes/dexhand021/r_f_link4_2.STL
- link r_f_link4_2_1: mass 0.0010001 -> 0.0009340644343591204; geometry collision mesh filename=../meshes/dexhand021/r_f_link4_2_1.STL; visual mesh filename=../meshes/dexhand021/r_f_link4_2_1.STL
- link r_f_link4_2_2: mass 0.0010001 -> 0.002679962972544183; geometry collision mesh filename=../meshes/dexhand021/r_f_link4_2_2.STL; visual mesh filename=../meshes/dexhand021/r_f_link4_2_2.STL
- link r_f_link4_3: mass 0.0035515 -> 0.0033203328984136053; geometry collision mesh filename=../meshes/dexhand021/r_f_link4_3.STL; visual mesh filename=../meshes/dexhand021/r_f_link4_3.STL
- link r_f_link4_3_1: mass 0.00053481 -> 0.000499830382166977; geometry collision mesh filename=../meshes/dexhand021/r_f_link4_3_1.STL; visual mesh filename=../meshes/dexhand021/r_f_link4_3_1.STL
- link r_f_link4_3_2: mass 0.00099236 -> 0.0009265838824928253; geometry collision mesh filename=../meshes/dexhand021/r_f_link4_3_2.STL; visual mesh filename=../meshes/dexhand021/r_f_link4_3_2.STL
- link r_f_link4_4: mass 0.0046613 -> 0.004352952819355013; geometry collision mesh filename=../meshes/dexhand021/r_f_link4_4.STL; visual mesh filename=../meshes/dexhand021/r_f_link4_4.STL
- link r_f_link4_4_1: mass 0.00041733 -> 0.00038943301930773646; geometry collision mesh filename=../meshes/dexhand021/r_f_link4_4_1.STL; visual mesh filename=../meshes/dexhand021/r_f_link4_4_1.STL
- link r_f_link4_4_2: mass 0.0110157 -> 0.0019468121676849014; geometry collision mesh filename=../meshes/dexhand021/r_f_link4_4_2.STL; visual mesh filename=../meshes/dexhand021/r_f_link4_4_2.STL
- link r_f_link5_1: mass 0.003769 -> 0.003518579086791241; geometry collision mesh filename=../meshes/dexhand021/r_f_link5_1.STL; visual mesh filename=../meshes/dexhand021/r_f_link5_1.STL
- link r_f_link5_2: mass 0.0053385 -> 0.004989367448655121; geometry collision mesh filename=../meshes/dexhand021/r_f_link5_2.STL; visual mesh filename=../meshes/dexhand021/r_f_link5_2.STL
- link r_f_link5_2_1: mass 0.00100007240206559 -> 0.0009340644343591205; geometry collision mesh filename=../meshes/dexhand021/r_f_link5_2_1.STL; visual mesh filename=../meshes/dexhand021/r_f_link5_2_1.STL
- link r_f_link5_2_2: mass 0.0028758 -> 0.002679962972544193; geometry collision mesh filename=../meshes/dexhand021/r_f_link5_2_2.STL; visual mesh filename=../meshes/dexhand021/r_f_link5_2_2.STL
- link r_f_link5_3: mass 0.0035515 -> 0.003320332898413456; geometry collision mesh filename=../meshes/dexhand021/r_f_link5_3.STL; visual mesh filename=../meshes/dexhand021/r_f_link5_3.STL
- link r_f_link5_3_1: mass 0.00053481 -> 0.0004998303821669769; geometry collision mesh filename=../meshes/dexhand021/r_f_link5_3_1.STL; visual mesh filename=../meshes/dexhand021/r_f_link5_3_1.STL
- link r_f_link5_3_2: mass 0.0028758 -> 0.0009265838824928253; geometry collision mesh filename=../meshes/dexhand021/r_f_link5_3_2.STL; visual mesh filename=../meshes/dexhand021/r_f_link5_3_2.STL
- link r_f_link5_4: mass 0.0046613 -> 0.004352952855182437; geometry collision mesh filename=../meshes/dexhand021/r_f_link5_4.STL; visual mesh filename=../meshes/dexhand021/r_f_link5_4.STL
- link r_f_link5_4_1: mass 0.00041733 -> 0.0003894330192680039; geometry collision mesh filename=../meshes/dexhand021/r_f_link5_4_1.STL; visual mesh filename=../meshes/dexhand021/r_f_link5_4_1.STL
- link r_f_link5_4_2: mass 0.0110157 -> 0.0019468121678303657; geometry collision mesh filename=../meshes/dexhand021/r_f_link5_4_2.STL; visual mesh filename=../meshes/dexhand021/r_f_link5_4_2.STL
- link r_p_link0: mass 0.13795 -> 0.4581543554912673; geometry collision mesh filename=../meshes/dexhand021/r_p_link0.STL; visual mesh filename=../meshes/dexhand021/r_p_link0.STL
- link r_p_link1: mass 0.027214 -> 0.08395173603509726; geometry collision mesh filename=../meshes/dexhand021/r_p_link1.STL; visual mesh filename=../meshes/dexhand021/r_p_link1.STL
- link r_p_link2: mass 0.023927 -> 0.07899657199227124; geometry collision mesh filename=../meshes/dexhand021/r_p_link2.STL; visual mesh filename=../meshes/dexhand021/r_p_link2.STL
- link r_p_link3: mass 0.01334 -> 0.044023395748120794; geometry collision mesh filename=../meshes/dexhand021/r_p_link3.STL; visual mesh filename=../meshes/dexhand021/r_p_link3.STL
- link r_p_link4: mass 0.025026 -> 0.08245656201270479; geometry collision mesh filename=../meshes/dexhand021/r_p_link4.STL; visual mesh filename=../meshes/dexhand021/r_p_link4.STL
- link r_p_link5: mass 0.0068413 -> 0.022516997147359073; geometry collision mesh filename=../meshes/dexhand021/r_p_link5.STL; visual mesh filename=../meshes/dexhand021/r_p_link5.STL
- link r_p_link6: mass 0.036663 -> 0.11253371281264385; geometry collision mesh filename=../meshes/dexhand021/r_p_link6.STL; visual mesh filename=../meshes/dexhand021/r_p_link6.STL

File: urdf/dexhand021_right_simplified.urdf (robot description, URDF)
Before this commit: robot dexhand021_right_simplified, 26 links, 25 joints
Links:
- link r_f_link1_1: mass 0.0055264 -> 0.004409963237919953; geometry collision mesh filename=../meshes/dexhand021_simplified/r_f_link1_1.STL; visual mesh filename=../meshes/dexhand021_simplified/r_f_link1_1.STL
- link r_f_link1_2: mass 0.012462 -> 0.009952224489361963; geometry collision mesh filename=../meshes/dexhand021_simplified/r_f_link1_2.STL; visual mesh filename=../meshes/dexhand021_simplified/r_f_link1_2.STL
- link r_f_link1_3: mass 0.005726 -> 0.004573330448687783; geometry collision mesh filename=../meshes/dexhand021_simplified/r_f_link1_3.STL; visual mesh filename=../meshes/dexhand021_simplified/r_f_link1_3.STL
- link r_f_link1_4: mass 0.0051136 -> 0.0061592845660588934; geometry collision mesh filename=../meshes/dexhand021_simplified/r_f_link1_4.STL; visual mesh filename=../meshes/dexhand021_simplified/r_f_link1_4.STL
- link r_f_link2_1: mass 0.0051273 -> 0.00409703693716023; geometry collision mesh filename=../meshes/dexhand021_simplified/r_f_link2_1.STL; visual mesh filename=../meshes/dexhand021_simplified/r_f_link2_1.STL
- link r_f_link2_2: mass 0.011802 -> 0.009428397870928118; geometry collision mesh filename=../meshes/dexhand021_simplified/r_f_link2_2.STL; visual mesh filename=../meshes/dexhand021_simplified/r_f_link2_2.STL
- link r_f_link2_3: mass 0.005726 -> 0.004573330342568089; geometry collision mesh filename=../meshes/dexhand021_simplified/r_f_link2_3.STL; visual mesh filename=../meshes/dexhand021_simplified/r_f_link2_3.STL
- link r_f_link2_4: mass 0.0051136 -> 0.006159284595780522; geometry collision mesh filename=../meshes/dexhand021_simplified/r_f_link2_4.STL; visual mesh filename=../meshes/dexhand021_simplified/r_f_link2_4.STL
- link r_f_link3_1: mass 0.0051273 -> 0.004097039690946969; geometry collision mesh filename=../meshes/dexhand021_simplified/r_f_link3_1.STL; visual mesh filename=../meshes/dexhand021_simplified/r_f_link3_1.STL
- link r_f_link3_2: mass 0.011802 -> 0.009428397870928118; geometry collision mesh filename=../meshes/dexhand021_simplified/r_f_link3_2.STL; visual mesh filename=../meshes/dexhand021_simplified/r_f_link3_2.STL
- link r_f_link3_3: mass 0.005726 -> 0.004573330342515683; geometry collision mesh filename=../meshes/dexhand021_simplified/r_f_link3_3.STL; visual mesh filename=../meshes/dexhand021_simplified/r_f_link3_3.STL
- link r_f_link3_4: mass 0.0051136 -> 0.006159284595780522; geometry collision mesh filename=../meshes/dexhand021_simplified/r_f_link3_4.STL; visual mesh filename=../meshes/dexhand021_simplified/r_f_link3_4.STL
- link r_f_link4_1: mass 0.0051273 -> 0.004097040417879458; geometry collision mesh filename=../meshes/dexhand021_simplified/r_f_link4_1.STL; visual mesh filename=../meshes/dexhand021_simplified/r_f_link4_1.STL
- link r_f_link4_2: mass 0.011802 -> 0.009428397870928114; geometry collision mesh filename=../meshes/dexhand021_simplified/r_f_link4_2.STL; visual mesh filename=../meshes/dexhand021_simplified/r_f_link4_2.STL
- link r_f_link4_3: mass 0.005726 -> 0.00457333034240358; geometry collision mesh filename=../meshes/dexhand021_simplified/r_f_link4_3.STL; visual mesh filename=../meshes/dexhand021_simplified/r_f_link4_3.STL
- link r_f_link4_4: mass 0.0051136 -> 0.006159284595780522; geometry collision mesh filename=../meshes/dexhand021_simplified/r_f_link4_4.STL; visual mesh filename=../meshes/dexhand021_simplified/r_f_link4_4.STL
- link r_f_link5_1: mass 0.003769 -> 0.004097034606160823; geometry collision mesh filename=../meshes/dexhand021_simplified/r_f_link5_1.STL; visual mesh filename=../meshes/dexhand021_simplified/r_f_link5_1.STL
- link r_f_link5_2: mass 0.011802 -> 0.009428397870928114; geometry collision mesh filename=../meshes/dexhand021_simplified/r_f_link5_2.STL; visual mesh filename=../meshes/dexhand021_simplified/r_f_link5_2.STL
- link r_f_link5_3: mass 0.005726 -> 0.004573330342463683; geometry collision mesh filename=../meshes/dexhand021_simplified/r_f_link5_3.STL; visual mesh filename=../meshes/dexhand021_simplified/r_f_link5_3.STL
- link r_f_link5_4: mass 0.0051136 -> 0.006159284595780522; geometry collision mesh filename=../meshes/dexhand021_simplified/r_f_link5_4.STL; visual mesh filename=../meshes/dexhand021_simplified/r_f_link5_4.STL
- link right_hand_base: mass 0.39703 -> 0.883463360898785; geometry collision mesh filename=../meshes/dexhand021_simplified/right_hand_base.STL; visual mesh filename=../meshes/dexhand021_simplified/right_hand_base.STL

Commit message: refactor(urdf): rename joint for consistency
Renamed joint "l_a_joint1_1" to "l_f_joint1_1" to maintain naming
consistency across the URDF file. This change helps in better
understanding and managing the joint hierarchy.

File: urdf/dexhand021_left.urdf (robot description, URDF)
Before this commit: robot dexhand021_left, 63 links, 62 joints
Joints:
- removed joint l_a_joint1_1
- added joint l_f_joint1_1: type revolute, parent l_p_link0, child l_f_link1_1, origin xyz=-0.023855 -0.031204 0.27607 rpy=0 -0.15197 -2.8876, axis 0 0.26521 0.96419, limit lower=0 upper=2.2 effort=10 velocity=1.5
