Commit message: Add fingertip pads and improve positioning of fingertips
🤖 Generated with [Claude Code](https://claude.ai/code)

Co-Authored-By: Claude <noreply@anthropic.com>

File: urdf/dexhand021_left.urdf (robot description, URDF)
Before this commit: robot dexhand021_left, 63 links, 62 joints
Links:
- added link l_f_link1_pad, mass 0.001; collision sphere radius=0.002; visual sphere radius=0.002
- added link l_f_link2_pad, mass 0.001; collision sphere radius=0.002; visual sphere radius=0.002
- added link l_f_link3_pad, mass 0.001; collision sphere radius=0.002; visual sphere radius=0.002
- added link l_f_link4_pad, mass 0.001; collision sphere radius=0.002; visual sphere radius=0.002
- added link l_f_link5_pad, mass 0.001; collision sphere radius=0.002; visual sphere radius=0.002
Joints:
- added joint l_f_joint1_pad: type fixed, parent l_f_link1_4, child l_f_link1_pad, origin xyz=0.026 0.003 0 rpy=0 0 0
- added joint l_f_joint2_pad: type fixed, parent l_f_link2_4, child l_f_link2_pad, origin xyz=0.026 0.003 0 rpy=0 0 0
- added joint l_f_joint3_pad: type fixed, parent l_f_link3_4, child l_f_link3_pad, origin xyz=0.026 0.003 0 rpy=0 0 0
- added joint l_f_joint4_pad: type fixed, parent l_f_link4_4, child l_f_link4_pad, origin xyz=0.026 0.003 0 rpy=0 0 0
- added joint l_f_joint5_pad: type fixed, parent l_f_link5_4, child l_f_link5_pad, origin xyz=0.026 0.003 0 rpy=0 0 0
- joint l_f_joint1_tip: origin xyz=0.02 0 0 rpy=0 0 0 -> xyz=0.035 -0.004 0 rpy=0 0 0
- joint l_f_joint2_tip: origin xyz=0.02 0 0 rpy=0 0 0 -> xyz=0.035 -0.004 0 rpy=0 0 0
- joint l_f_joint3_tip: origin xyz=0.02 0 0 rpy=0 0 0 -> xyz=0.035 -0.004 0 rpy=0 0 0
- joint l_f_joint4_tip: origin xyz=0.02 0 0 rpy=0 0 0 -> xyz=0.035 -0.004 0 rpy=0 0 0
- joint l_f_joint5_tip: origin xyz=0.02 0 0 rpy=0 0 0 -> xyz=0.035 -0.004 0 rpy=0 0 0

File: urdf/dexhand021_left_simplified.urdf (robot description, URDF)
Before this commit: robot dexhand021_left_simplified, 26 links, 25 joints
Links:
- added link l_f_link1_pad, mass 0.001; collision sphere radius=0.002; visual sphere radius=0.002
- added link l_f_link2_pad, mass 0.001; collision sphere radius=0.002; visual sphere radius=0.002
- added link l_f_link3_pad, mass 0.001; collision sphere radius=0.002; visual sphere radius=0.002
- added link l_f_link4_pad, mass 0.001; collision sphere radius=0.002; visual sphere radius=0.002
- added link l_f_link5_pad, mass 0.001; collision sphere radius=0.002; visual sphere radius=0.002
Joints:
- added joint l_f_joint1_pad: type fixed, parent l_f_link1_4, child l_f_link1_pad, origin xyz=0.026 0.003 0 rpy=0 0 0
- added joint l_f_joint2_pad: type fixed, parent l_f_link2_4, child l_f_link2_pad, origin xyz=0.026 0.003 0 rpy=0 0 0
- added joint l_f_joint3_pad: type fixed, parent l_f_link3_4, child l_f_link3_pad, origin xyz=0.026 0.003 0 rpy=0 0 0
- added joint l_f_joint4_pad: type fixed, parent l_f_link4_4, child l_f_link4_pad, origin xyz=0.026 0.003 0 rpy=0 0 0
- added joint l_f_joint5_pad: type fixed, parent l_f_link5_4, child l_f_link5_pad, origin xyz=0.026 0.003 0 rpy=0 0 0
- joint l_f_joint1_tip: origin xyz=0.02 0 0 rpy=0 0 0 -> xyz=0.035 -0.004 0 rpy=0 0 0
- joint l_f_joint2_tip: origin xyz=0.02 0 0 rpy=0 0 0 -> xyz=0.035 -0.004 0 rpy=0 0 0
- joint l_f_joint3_tip: origin xyz=0.02 0 0 rpy=0 0 0 -> xyz=0.035 -0.004 0 rpy=0 0 0
- joint l_f_joint4_tip: origin xyz=0.02 0 0 rpy=0 0 0 -> xyz=0.035 -0.004 0 rpy=0 0 0
- joint l_f_joint5_tip: origin xyz=0.02 0 0 rpy=0 0 0 -> xyz=0.035 -0.004 0 rpy=0 0 0

File: urdf/dexhand021_right.urdf (robot description, URDF)
Before this commit: robot dexhand021_right, 63 links, 62 joints
Links:
- added link r_f_link1_pad, mass 0.001; collision sphere radius=0.002; visual sphere radius=0.002
- added link r_f_link2_pad, mass 0.001; collision sphere radius=0.002; visual sphere radius=0.002
- added link r_f_link3_pad, mass 0.001; collision sphere radius=0.002; visual sphere radius=0.002
- added link r_f_link4_pad, mass 0.001; collision sphere radius=0.002; visual sphere radius=0.002
- added link r_f_link5_pad, mass 0.001; collision sphere radius=0.002; visual sphere radius=0.002
Joints:
- added joint r_f_joint1_pad: type fixed, parent r_f_link1_4, child r_f_link1_pad, origin xyz=0.026 0.003 0 rpy=0 0 0
- added joint r_f_joint2_pad: type fixed, parent r_f_link2_4, child r_f_link2_pad, origin xyz=0.026 0.003 0 rpy=0 0 0
- added joint r_f_joint3_pad: type fixed, parent r_f_link3_4, child r_f_link3_pad, origin xyz=0.026 0.003 0 rpy=0 0 0
- added joint r_f_joint4_pad: type fixed, parent r_f_link4_4, child r_f_link4_pad, origin xyz=0.026 0.003 0 rpy=0 0 0
- added joint r_f_joint5_pad: type fixed, parent r_f_link5_4, child r_f_link5_pad, origin xyz=0.026 0.003 0 rpy=0 0 0
- joint r_f_joint1_tip: origin xyz=0.02 0 0 rpy=0 0 0 -> xyz=0.035 -0.004 0 rpy=0 0 0
- joint r_f_joint2_tip: origin xyz=0.02 0 0 rpy=0 0 0 -> xyz=0.035 -0.004 0 rpy=0 0 0
- joint r_f_joint3_tip: origin xyz=0.02 0 0 rpy=0 0 0 -> xyz=0.035 -0.004 0 rpy=0 0 0
- joint r_f_joint4_tip: origin xyz=0.02 0 0 rpy=0 0 0 -> xyz=0.035 -0.004 0 rpy=0 0 0
- joint r_f_joint5_tip: origin xyz=0.02 0 0 rpy=0 0 0 -> xyz=0.035 -0.004 0 rpy=0 0 0

File: urdf/dexhand021_right_simplified.urdf (robot description, URDF)
Before this commit: robot dexhand021_right_simplified, 26 links, 25 joints
Links:
- added link r_f_link1_pad, mass 0.001; collision sphere radius=0.002; visual sphere radius=0.002
- added link r_f_link2_pad, mass 0.001; collision sphere radius=0.002; visual sphere radius=0.002
- added link r_f_link3_pad, mass 0.001; collision sphere radius=0.002; visual sphere radius=0.002
- added link r_f_link4_pad, mass 0.001; collision sphere radius=0.002; visual sphere radius=0.002
- added link r_f_link5_pad, mass 0.001; collision sphere radius=0.002; visual sphere radius=0.002
Joints:
- added joint r_f_joint1_pad: type fixed, parent r_f_link1_4, child r_f_link1_pad, origin xyz=0.026 0.003 0 rpy=0 0 0
- added joint r_f_joint2_pad: type fixed, parent r_f_link2_4, child r_f_link2_pad, origin xyz=0.026 0.003 0 rpy=0 0 0
- added joint r_f_joint3_pad: type fixed, parent r_f_link3_4, child r_f_link3_pad, origin xyz=0.026 0.003 0 rpy=0 0 0
- added joint r_f_joint4_pad: type fixed, parent r_f_link4_4, child r_f_link4_pad, origin xyz=0.026 0.003 0 rpy=0 0 0
- added joint r_f_joint5_pad: type fixed, parent r_f_link5_4, child r_f_link5_pad, origin xyz=0.026 0.003 0 rpy=0 0 0
- joint r_f_joint1_tip: origin xyz=0.02 0 0 rpy=0 0 0 -> xyz=0.035 -0.004 0 rpy=0 0 0
- joint r_f_joint2_tip: origin xyz=0.02 0 0 rpy=0 0 0 -> xyz=0.035 -0.004 0 rpy=0 0 0
- joint r_f_joint3_tip: origin xyz=0.02 0 0 rpy=0 0 0 -> xyz=0.035 -0.004 0 rpy=0 0 0
- joint r_f_joint4_tip: origin xyz=0.02 0 0 rpy=0 0 0 -> xyz=0.035 -0.004 0 rpy=0 0 0
- joint r_f_joint5_tip: origin xyz=0.02 0 0 rpy=0 0 0 -> xyz=0.035 -0.004 0 rpy=0 0 0

Commit message: feat: update fingerpads from spheres to thin boxes
- Changed fingerpads from small spheres to thin rectangular pads
- Adjusted positioning and orientation for better contact simulation
- Updated documentation with explanation of fingertips and fingerpads
- Added documentation in English and Chinese

🤖 Generated with [Claude Code](https://claude.ai/code)

Co-Authored-By: Claude <noreply@anthropic.com>

File: urdf/dexhand021_left.urdf (robot description, URDF)
Before this commit: robot dexhand021_left, 68 links, 67 joints
Links:
- link l_f_link1_pad: geometry collision box size=0.012 0.001 0.006; visual box size=0.012 0.001 0.006
- link l_f_link2_pad: geometry collision box size=0.012 0.001 0.006; visual box size=0.012 0.001 0.006
- link l_f_link3_pad: geometry collision box size=0.012 0.001 0.006; visual box size=0.012 0.001 0.006
- link l_f_link4_pad: geometry collision box size=0.012 0.001 0.006; visual box size=0.012 0.001 0.006
- link l_f_link5_pad: geometry collision box size=0.012 0.001 0.006; visual box size=0.012 0.001 0.006
Joints:
- joint l_f_joint1_pad: origin xyz=0.026 0.003 0 rpy=0 0 0 -> xyz=0.026 0.0025 0.001 rpy=0 0 0
- joint l_f_joint2_pad: origin xyz=0.026 0.003 0 rpy=0 0 0 -> xyz=0.026 0.0025 0.000 rpy=0 0 0
- joint l_f_joint3_pad: origin xyz=0.026 0.003 0 rpy=0 0 0 -> xyz=0.026 0.0025 0.000 rpy=0 0 0
- joint l_f_joint4_pad: origin xyz=0.026 0.003 0 rpy=0 0 0 -> xyz=0.026 0.0025 0.000 rpy=0 0 0
- joint l_f_joint5_pad: origin xyz=0.026 0.003 0 rpy=0 0 0 -> xyz=0.026 0.0025 0.000 rpy=0 0 0

File: urdf/dexhand021_left_simplified.urdf (robot description, URDF)
Before this commit: robot dexhand021_left_simplified, 31 links, 30 joints
Links:
- link l_f_link1_pad: geometry collision box size=0.012 0.001 0.006; visual box size=0.012 0.001 0.006
- link l_f_link2_pad: geometry collision box size=0.012 0.001 0.006; visual box size=0.012 0.001 0.006
- link l_f_link3_pad: geometry collision box size=0.012 0.001 0.006; visual box size=0.012 0.001 0.006
- link l_f_link4_pad: geometry collision box size=0.012 0.001 0.006; visual box size=0.012 0.001 0.006
- link l_f_link5_pad: geometry collision box size=0.012 0.001 0.006; visual box size=0.012 0.001 0.006
Joints:
- joint l_f_joint1_pad: origin xyz=0.026 0.003 0 rpy=0 0 0 -> xyz=0.026 0.0025 0.001 rpy=0 0 0
- joint l_f_joint2_pad: origin xyz=0.026 0.003 0 rpy=0 0 0 -> xyz=0.026 0.0025 0.000 rpy=0 0 0
- joint l_f_joint3_pad: origin xyz=0.026 0.003 0 rpy=0 0 0 -> xyz=0.026 0.0025 0.000 rpy=0 0 0
- joint l_f_joint4_pad: origin xyz=0.026 0.003 0 rpy=0 0 0 -> xyz=0.026 0.0025 0.000 rpy=0 0 0
- joint l_f_joint5_pad: origin xyz=0.026 0.003 0 rpy=0 0 0 -> xyz=0.026 0.0025 0.000 rpy=0 0 0

File: urdf/dexhand021_right.urdf (robot description, URDF)
Before this commit: robot dexhand021_right, 68 links, 67 joints
Links:
- link r_f_link1_pad: geometry collision box size=0.012 0.001 0.006; visual box size=0.012 0.001 0.006
- link r_f_link2_pad: geometry collision box size=0.012 0.001 0.006; visual box size=0.012 0.001 0.006
- link r_f_link3_pad: geometry collision box size=0.012 0.001 0.006; visual box size=0.012 0.001 0.006
- link r_f_link4_pad: geometry collision box size=0.012 0.001 0.006; visual box size=0.012 0.001 0.006
- link r_f_link5_pad: geometry collision box size=0.012 0.001 0.006; visual box size=0.012 0.001 0.006
Joints:
- joint r_f_joint1_pad: origin xyz=0.026 0.003 0 rpy=0 0 0 -> xyz=0.026 0.0025 0.001 rpy=0 0 0
- joint r_f_joint2_pad: origin xyz=0.026 0.003 0 rpy=0 0 0 -> xyz=0.026 0.0025 0.000 rpy=0 0 0
- joint r_f_joint3_pad: origin xyz=0.026 0.003 0 rpy=0 0 0 -> xyz=0.026 0.0025 0.000 rpy=0 0 0
- joint r_f_joint4_pad: origin xyz=0.026 0.003 0 rpy=0 0 0 -> xyz=0.026 0.0025 0.000 rpy=0 0 0
- joint r_f_joint5_pad: origin xyz=0.026 0.003 0 rpy=0 0 0 -> xyz=0.026 0.0025 0.000 rpy=0 0 0

File: urdf/dexhand021_right_simplified.urdf (robot description, URDF)
Before this commit: robot dexhand021_right_simplified, 31 links, 30 joints
Links:
- link r_f_link1_pad: geometry collision box size=0.012 0.001 0.006; visual box size=0.012 0.001 0.006
- link r_f_link2_pad: geometry collision box size=0.012 0.001 0.006; visual box size=0.012 0.001 0.006
- link r_f_link3_pad: geometry collision box size=0.012 0.001 0.006; visual box size=0.012 0.001 0.006
- link r_f_link4_pad: geometry collision box size=0.012 0.001 0.006; visual box size=0.012 0.001 0.006
- link r_f_link5_pad: geometry collision box size=0.012 0.001 0.006; visual box size=0.012 0.001 0.006
Joints:
- joint r_f_joint1_pad: origin xyz=0.026 0.003 0 rpy=0 0 0 -> xyz=0.026 0.0025 -0.001 rpy=0 0 0
- joint r_f_joint2_pad: origin xyz=0.026 0.003 0 rpy=0 0 0 -> xyz=0.026 0.0025 0.000 rpy=0 0 0
- joint r_f_joint3_pad: origin xyz=0.026 0.003 0 rpy=0 0 0 -> xyz=0.026 0.0025 0.000 rpy=0 0 0
- joint r_f_joint4_pad: origin xyz=0.026 0.003 0 rpy=0 0 0 -> xyz=0.026 0.0025 0.000 rpy=0 0 0
- joint r_f_joint5_pad: origin xyz=0.026 0.003 0 rpy=0 0 0 -> xyz=0.026 0.0025 0.000 rpy=0 0 0

Commit message: fix(urdf): correct fingerpad rotation by moving it to joint instead of link
🤖 Generated with [Claude Code](https://claude.ai/code)

Co-Authored-By: Claude <noreply@anthropic.com>

File: urdf/dexhand021_left.urdf (robot description, URDF)
Before this commit: robot dexhand021_left, 68 links, 67 joints
Joints:
- joint l_f_joint1_pad: origin xyz=0.026 0.0025 0.001 rpy=0 0 0 -> xyz=0.026 0.0025 0.001 rpy=0 0 -0.45
- joint l_f_joint2_pad: origin xyz=0.026 0.0025 0.000 rpy=0 0 0 -> xyz=0.026 0.0025 0.000 rpy=0 0 -0.45
- joint l_f_joint3_pad: origin xyz=0.026 0.0025 0.000 rpy=0 0 0 -> xyz=0.026 0.0025 0.000 rpy=0 0 -0.45
- joint l_f_joint4_pad: origin xyz=0.026 0.0025 0.000 rpy=0 0 0 -> xyz=0.026 0.0025 0.000 rpy=0 0 -0.45
- joint l_f_joint5_pad: origin xyz=0.026 0.0025 0.000 rpy=0 0 0 -> xyz=0.026 0.0025 0.000 rpy=0 0 -0.45

File: urdf/dexhand021_left_simplified.urdf (robot description, URDF)
Before this commit: robot dexhand021_left_simplified, 31 links, 30 joints
Joints:
- joint l_f_joint1_pad: origin xyz=0.026 0.0025 0.001 rpy=0 0 0 -> xyz=0.026 0.0025 0.001 rpy=0 0 -0.45
- joint l_f_joint2_pad: origin xyz=0.026 0.0025 0.000 rpy=0 0 0 -> xyz=0.026 0.0025 0.000 rpy=0 0 -0.45
- joint l_f_joint3_pad: origin xyz=0.026 0.0025 0.000 rpy=0 0 0 -> xyz=0.026 0.0025 0.000 rpy=0 0 -0.45
- joint l_f_joint4_pad: origin xyz=0.026 0.0025 0.000 rpy=0 0 0 -> xyz=0.026 0.0025 0.000 rpy=0 0 -0.45
- joint l_f_joint5_pad: origin xyz=0.026 0.0025 0.000 rpy=0 0 0 -> xyz=0.026 0.0025 0.000 rpy=0 0 -0.45

File: urdf/dexhand021_right.urdf (robot description, URDF)
Before this commit: robot dexhand021_right, 68 links, 67 joints
Joints:
- joint r_f_joint1_pad: origin xyz=0.026 0.0025 0.001 rpy=0 0 0 -> xyz=0.026 0.0025 0.001 rpy=0 0 -0.45
- joint r_f_joint2_pad: origin xyz=0.026 0.0025 0.000 rpy=0 0 0 -> xyz=0.026 0.0025 0.000 rpy=0 0 -0.45
- joint r_f_joint3_pad: origin xyz=0.026 0.0025 0.000 rpy=0 0 0 -> xyz=0.026 0.0025 0.000 rpy=0 0 -0.45
- joint r_f_joint4_pad: origin xyz=0.026 0.0025 0.000 rpy=0 0 0 -> xyz=0.026 0.0025 0.000 rpy=0 0 -0.45
- joint r_f_joint5_pad: origin xyz=0.026 0.0025 0.000 rpy=0 0 0 -> xyz=0.026 0.0025 0.000 rpy=0 0 -0.45

File: urdf/dexhand021_right_simplified.urdf (robot description, URDF)
Before this commit: robot dexhand021_right_simplified, 31 links, 30 joints
Joints:
- joint r_f_joint1_pad: origin xyz=0.026 0.0025 -0.001 rpy=0 0 0 -> xyz=0.026 0.0025 -0.001 rpy=0 0 -0.45
- joint r_f_joint2_pad: origin xyz=0.026 0.0025 0.000 rpy=0 0 0 -> xyz=0.026 0.0025 0.000 rpy=0 0 -0.45
- joint r_f_joint3_pad: origin xyz=0.026 0.0025 0.000 rpy=0 0 0 -> xyz=0.026 0.0025 0.000 rpy=0 0 -0.45
- joint r_f_joint4_pad: origin xyz=0.026 0.0025 0.000 rpy=0 0 0 -> xyz=0.026 0.0025 0.000 rpy=0 0 -0.45
- joint r_f_joint5_pad: origin xyz=0.026 0.0025 0.000 rpy=0 0 0 -> xyz=0.026 0.0025 0.000 rpy=0 0 -0.45
